Commit message: planning scene v2

File: franka_mis_description/urdf/table_mis.xacro (robot description, xacro)
@@ -3,12 +3,12 @@
     <xacro:arg name="arm_id" default="panda" />
     <xacro:include filename="$(find franka_mis_description)/urdf/table_mis_macro.xacro"/>
+    <xacro:table_mis prefix=""/>
     <!-- <xacro:include filename="$(find franka_description)/robots/utils.xacro"/>
     <xacro:include filename="$(find franka_description)/robots/panda_arm.xacro"/>
     <xacro:panda_arm arm_id="$(arg arm_id)" safety_distance="0.03"/>
-    <xacro:table_mis prefix=""/> -->
     <joint name="table_panda_joint" type="fixed">
         <origin xyz="0 0 0" rpy="0 0 -1.57" />
         <parent link="plank" />
         <child  link="$(arg arm_id)_link0" />
-    </joint>
+    </joint> -->
 </robot>

Commit message: v2: own FK

File: franka_mis_description/urdf/table_mis.xacro (robot description, xacro)
@@ -4,5 +4,5 @@
     <xacro:include filename="$(find franka_mis_description)/urdf/table_mis_macro.xacro"/>
     <xacro:table_mis prefix=""/>
-    <!-- <xacro:include filename="$(find franka_description)/robots/utils.xacro"/>
+    <xacro:include filename="$(find franka_description)/robots/utils.xacro"/>
     <xacro:include filename="$(find franka_description)/robots/panda_arm.xacro"/>
     <xacro:panda_arm arm_id="$(arg arm_id)" safety_distance="0.03"/>
@@ -11,4 +11,4 @@
         <parent link="plank" />
         <child  link="$(arg arm_id)_link0" />
-    </joint> -->
+    </joint>
 </robot>

Commit message: add chobot

File: franka_mis_description/urdf/table_mis.xacro (robot description, xacro)
@@ -2,9 +2,15 @@
 <robot name="franka_mis" xmlns:xacro="http://www.ros.org/wiki/xacro">
     <xacro:arg name="arm_id" default="panda" />
+    <!-- Add table scene -->
     <xacro:include filename="$(find franka_mis_description)/urdf/table_mis_macro.xacro"/>
     <xacro:table_mis prefix=""/>
+    <!-- Add chobot -->
+    <xacro:include filename="$(find franka_mis_description)/urdf/chobot_mis_macro.xacro"/>
+    <xacro:chobot_mis prefix=""/>
+    <!-- Add Panda -->
     <xacro:include filename="$(find franka_description)/robots/utils.xacro"/>
     <xacro:include filename="$(find franka_description)/robots/panda_arm.xacro"/>
     <xacro:panda_arm arm_id="$(arg arm_id)" safety_distance="0.03"/>
+    <!-- Create joints -->
     <joint name="table_panda_joint" type="fixed">
         <origin xyz="0 0 0" rpy="0 0 -1.57" />
@@ -12,3 +18,8 @@
         <child  link="$(arg arm_id)_link0" />
     </joint>
+    <joint name="panda_chobot_joint" type="fixed">
+        <origin xyz="0 0 0" rpy="0 0 -1.57" />
+        <parent link="$(arg arm_id)_link8" />
+        <child  link="chobot_base" />
+    </joint>
 </robot>
